File: SolarLights_Lite/kicad_current/SolarLights_Lite_Current.kicad_sch (KiCad schematic)
At the start: 24 parts, among them J1 PV in, J2 LED string, M1 TP4056 + DW01A, M2 BTE13-010A - int. 8 MHz, M3 Wemos D1 Mini, Q2 2N3904, SW1 test, U0 5 V reg - TBD, U3 3V3 tel. - HL802A cand.

Commit message: Refine v0.5 live project documentation
Parts:
- M3: Note ESPHome, hourly deep sleep; onboard regulator removed -> ESPHome v0.5 development UART; always-on; onboard regulator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
- Q2: Note telemetry status inverter -> development UART inverter
Connections:
- net at Q2.2 (C), R10.1: now also M3.D6; no longer M3.D5
- net at R8.1: now also M2.D1 (D1 TX); no longer M2.D8 (D8 lights)
Changed lines of the file:
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@@
   (title_block
     (title "Solar Front Lights - Lite (current build)")
-    (date "2026-09-21")
-    (rev "0.4b")
+    (date "27-Sep-2026")
+    (rev "0.5")
     (company "AJC & Co")
-    (comment 1 "Flow: panel -> U0 (TBD 5V reg) -> TP4056 -> battery rail -> Pro Mini, direct-drive LED, D1 Mini")
-    (comment 2 "21 Sep 2026: Q1/R6/R7/F1 removed - D9 drives R3 (47R) directly, approx 15 mA @3.7 V. U0 still TBD; U3 candidate = TPS63802/HL802A breakout (not U0 - 5.5V input ceiling too low for panel Voc).")
+    (comment 1 "Flow: panel -> U0 -> TP4056 -> battery rail -> Pro Mini, direct-drive LED and D1 Mini development telemetry")
+    (comment 2 "v0.5: Arduino D1/TX -> R8/Q2/R10 -> D1 Mini D6 (inverted 9600-baud UART). D8 and D5 are open in the development profile.")
   )
   (text "1  Panel in - U0 (TBD 5 V reg) - TP4056 charger - cells" (at 20 24 0) (effects (font (size 2.54 2.54) (thickness 0.508) bold) (justify left bottom)))
@@
   (wire (pts (xy 317.54 114.19) (xy 330.00 114.19)) (stroke (width 0) (type default)))
   (wire (pts (xy 330.00 114.19) (xy 365.00 114.19)) (stroke (width 0) (type default)))
-  (wire (pts (xy 365.00 114.19) (xy 365.00 169.92)) (stroke (width 0) (type default)))
-  (wire (pts (xy 365.00 169.92) (xy 350.32 169.92)) (stroke (width 0) (type default)))
+  (wire (pts (xy 365.00 114.19) (xy 365.00 177.54)) (stroke (width 0) (type default)))
+  (wire (pts (xy 365.00 177.54) (xy 309.68 177.54)) (stroke (width 0) (type default)))
   (wire (pts (xy 309.68 172.46) (xy 305.00 172.46)) (stroke (width 0) (type default)))
   (wire (pts (xy 305.00 172.46) (xy 305.00 186.00)) (stroke (width 0) (type default)))
@@
   (no_connect (at 251.59 120.00))
   (no_connect (at 251.59 122.54))
-  (no_connect (at 309.68 177.54))
+  (no_connect (at 350.32 169.92))
   (symbol (lib_id "Connector_Generic:Conn_01x02") (at 30.00 45.00 180) (unit 1)
     (in_bom yes) (on_board yes) (dnp no)
@@
     (pin "A1")
     (pin "D9")
-    (pin "D8")
+    (pin "D1")
     (pin "D2")
     (pin "D10")
@@
     (property "Footprint" "" (at 295.00 130.00 0) (effects (font (size 1.27 1.27)) hide))
     (property "Datasheet" "~" (at 295.00 130.00 0) (effects (font (size 1.27 1.27)) hide))
-    (property "Note" "telemetry status inverter" (at 295.00 137.62 0) (effects (font (size 1.016 1.016)) (justify left)))
+    (property "Note" "development UART inverter" (at 295.00 137.62 0) (effects (font (size 1.016 1.016)) (justify left)))
     (pin "1")
     (pin "2")
@@
     (property "Footprint" "" (at 330.00 175.00 0) (effects (font (size 1.27 1.27)) hide))
     (property "Datasheet" "~" (at 330.00 175.00 0) (effects (font (size 1.27 1.27)) hide))
-    (property "Note" "ESPHome, hourly deep sleep; onboard regulator removed" (at 330.00 191.51 0) (effects (font (size 1.016 1.016)) (justify left)))
+    (property "Note" "ESPHome v0.5 development UART; always-on; onboard regulator removed" (at 330.00 191.51 0) (effects (font (size 1.016 1.016)) (justify left)))
     (pin "5V")
     (pin "G")

Commit message: Rework v0.5 schematic layout and documentation
Parts:
- M3: Note ESPHome v0.5 development UART; always-on; onboard regulator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 -> ESPHome v0.5 dev UART; always-on; onboard regulator removed
- Q2: Note development UART inverter -> dev UART inverter
- R10: Note pull-up to 3V3_TEL -> pull-up
- R9: Note base-emitter pulldown -> B-E pulldown
Connections:
- net 3V3_TEL: now also M3.5V, R10.2, U3.OUT+
- net VBAT: now reaches C2.1, C3.1, M2.VCC, R5.1, S1.2 (B), U3.IN+
- net BATT_BUS: now reaches FB1.1, FB2.1, M1.B+
- net PWM: now reaches M2.D9 (D9 PWM), R3.1
- net BATT-: now reaches BT1.2 (-), BT2.2 (-), M1.B- (B−)
- net BTN: now reaches M2.D2 (D2 btn), SW1.1
- net D1_D6: now reaches M3.D6, Q2.2 (C), R10.1
- net UART_TX: now reaches M2.D1 (D1 TX), R8.1
- no-connect marks 5 -> 6
Other:
- note added: "1 Solar input, charger & cells"
- note added: "1S2P - each cell fused off the charger B+ node. TP4056 CHRG not wired."
- note added: "2 Battery rail - fuse + service switch"
- note added: "3 LED output - direct pin drive"
- note added: "4 Controller - Pro Mini BTE13-010A"
- note added: "5 Telemetry - Wemos D1 Mini (development)"
- note added: "6 Telemetry 3.3 V supply"
- note added: "Arduino D1/TX -> inverted 9600-baud UART -> D6. D0-RST for deep-sleep wake."
- note added: "Light sensor (switched by D7)"
- note added: "Test button"
- note added: "VBAT feeds the Pro Mini, U3 and R5 by net label"
- note added: "no Q1 / R6 / R7 / F1 - D9 drives the string through R3"
- note removed: "1 Panel in - U0 (TBD 5 V reg) - TP4056 charger - cells"
- note removed: "2 Battery rail: fused 1S2P + service switch"
- note removed: "3 LED driver: direct drive, no MOSFET"
- note removed: "4 Arduino (BTE13-010A) - dusk/dawn, schedule, PWM"
- note removed: "5 Wemos D1 Mini - reports to Home Assistant"
- moved on the sheet: BT1, BT2, C2, C3, F2, FB1, FB2, J1, J2, M1, M3, Q2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

Commit message: docs(hardware): record as-built v0.5 wiring, R4 47k and bench power
- Treat the whole v0.5 circuit as built; the switched LDR is wired.
- R4 changed 100k -> 47k: at 100k the 30% dark threshold needed LDR > ~233k,
  so a dim-but-not-dark bench never confirmed dusk. Covered LDR now reads 9.1%.
- U0 marked as an open item (not fitted; bench uses a 5 V panel direct to M1).
- U3 TPS63802 at 3.3 V on VBAT_SYS; bench D1 runs on micro-USB with U3 OUT
  disconnected, production D1 runs from U3 only.
- Record ~12% slow WDT scheduler clock.
- Regenerate drawing sheets, assembly guide, A3 PDF and KiCad schematic/PDF.
- main.cpp: LDR_DARK comment only; firmware output unchanged.
Parts:
- M3: Note ESPHome v0.5 dev UART; always-on; onboard regulator removed -> ESPHome v0.5 dev UART; bench: micro-USB power, U3 OUT disco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
- R4: value 100k -> 47k
- U0: value 5 V reg - TBD -> 5 V reg - OPEN ITEM; Note module not yet selected - see BUILD_GUIDE.md -> open item: not fitted; bench 5 V panel direct to M1 - see B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
- U3: value 3V3 tel. - HL802A cand. -> 3V3 tel. - TPS63802; Note TPS63802/HL802A breakout, jumper=3.3V; candidate, not bench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 -> TPS63802/HL802A, 3.3V; OUT to D1 3V3 in production only
Changed lines of the file:
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@@
     (in_bom yes) (on_board yes) (dnp no)
     (property "Reference" "U0" (at 76.20 44.45 0) (effects (font (size 1.27 1.27))))
-    (property "Value" "5 V reg - TBD" (at 76.20 46.99 0) (effects (font (size 1.27 1.27))))
+    (property "Value" "5 V reg - OPEN ITEM" (at 76.20 46.99 0) (effects (font (size 1.27 1.27))))
     (property "Footprint" "" (at 76.20 53.34 0) (effects (font (size 1.27 1.27)) hide))
     (property "Datasheet" "~" (at 76.20 53.34 0) (effects (font (size 1.27 1.27)) hide))
-    (property "Note" "module not yet selected - see BUILD_GUIDE.md" (at 76.20 60.32 0) (effects (font (size 1.016 1.016) italic)))
+    (property "Note" "open item: not fitted; bench 5 V panel direct to M1 - see BUILD_GUIDE.md" (at 76.20 60.32 0) (effects (font (size 1.016 1.016) italic)))
     (pin "IN+")
     (pin "IN-")
@@
     (in_bom yes) (on_board yes) (dnp no)
     (property "Reference" "R4" (at 43.18 226.06 0) (effects (font (size 1.27 1.27)) (justify left)))
-    (property "Value" "100k" (at 43.18 228.60 0) (effects (font (size 1.27 1.27)) (justify left)))
+    (property "Value" "47k" (at 43.18 228.60 0) (effects (font (size 1.27 1.27)) (justify left)))
     (property "Footprint" "Resistor_THT:R_Axial_DIN0207_L6.3mm_D2.5mm_P10.16mm_Horizontal" (at 40.64 227.33 0) (effects (font (size 1.27 1.27)) hide))
     (property "Datasheet" "~" (at 40.64 227.33 0) (effects (font (size 1.27 1.27)) hide))
@@
     (property "Footprint" "" (at 325.12 167.64 0) (effects (font (size 1.27 1.27)) hide))
     (property "Datasheet" "~" (at 325.12 167.64 0) (effects (font (size 1.27 1.27)) hide))
-    (property "Note" "ESPHome v0.5 dev UART; always-on; onboard regulator removed" (at 325.12 177.16 0) (effects (font (size 1.016 1.016) italic)))
+    (property "Note" "ESPHome v0.5 dev UART; bench: micro-USB power, U3 OUT disconnected" (at 325.12 177.16 0) (effects (font (size 1.016 1.016) italic)))
     (pin "5V")
     (pin "D6")
@@
     (in_bom yes) (on_board yes) (dnp no)
     (property "Reference" "U3" (at 248.92 214.63 0) (effects (font (size 1.27 1.27))))
-    (property "Value" "3V3 tel. - HL802A cand." (at 248.92 217.17 0) (effects (font (size 1.27 1.27))))
+    (property "Value" "3V3 tel. - TPS63802" (at 248.92 217.17 0) (effects (font (size 1.27 1.27))))
     (property "Footprint" "" (at 248.92 223.52 0) (effects (font (size 1.27 1.27)) hide))
     (property "Datasheet" "~" (at 248.92 223.52 0) (effects (font (size 1.27 1.27)) hide))
-    (property "Note" "TPS63802/HL802A breakout, jumper=3.3V; candidate, not bench-qualified" (at 281.94 226.06 0) (effects (font (size 1.016 1.016) italic) (justify left)))
+    (property "Note" "TPS63802/HL802A, 3.3V; OUT to D1 3V3 in production only" (at 281.94 226.06 0) (effects (font (size 1.016 1.016) italic) (justify left)))
     (pin "IN+")
     (pin "IN-")
