File: hardware/kicad/SolarLights_Lite.kicad_sch (KiCad schematic)
At the start: 24 parts, among them J1 PV in, J2 LED string, M1 TP4056 + DW01A, M2 BTE13-010A - int. 8 MHz, M3 Wemos D1 Mini, Q2 2N3904, SW1 test, U0 5 V buck (Option B), U3 3V3 tel. - TPS63802

Commit message: feat(pcb): carrier Rev C with LDR trim, TEST button and box-header ISP
R3 56R, R4 22k + RV1 50k 3296W rheostat, on-board 6x6 TEST switch, sideways
ISP with optional DC3-6P box header, name and repo on silkscreen. Docs 01-13,
drawings, layouts, netlist, KiCad schematic and renders follow Rev C.
Parts:
- added RV1: 50k trim, Potentiometer_THT:Potentiometer_Bourns_3296W_Vertical, symbol Device:R_Potentiometer
- R3: value 47R -> 56R; Note low-power string only; model ~15 mA @3.7 V, 56R if >22 mA @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 -> low-power string only; model ~13 mA @3.7 V, 68R if >20 mA @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
- R4: value 47k -> 22k
- SW1: value test -> TEST
Connections:
- net GND: now also RV1.2, RV1.3; no longer R4.2
- new net: R4.2, RV1.1
Other:
- note added: "Light sensor (switched by D7), RV1 sets dusk"
- note removed: "Light sensor (switched by D7)"
- moved on the sheet: LDR1, R4
Changed lines of the file:
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@@
   (label "BTN" (at 129.54 162.56 0) (fields_autoplaced) (effects (font (size 1.27 1.27)) (justify left bottom)))
   (label "LDR_PWR" (at 129.54 165.10 0) (fields_autoplaced) (effects (font (size 1.27 1.27)) (justify left bottom)))
-  (label "LDR_PWR" (at 33.02 203.20 180) (fields_autoplaced) (effects (font (size 1.27 1.27)) (justify right bottom)))
-  (label "LDR_SENSE" (at 48.26 218.44 0) (fields_autoplaced) (effects (font (size 1.27 1.27)) (justify left bottom)))
-  (text "Light sensor (switched by D7)" (at 20.32 195.58 0) (effects (font (size 1.27 1.27) (thickness 0.1524)) (justify left bottom)))
+  (label "LDR_PWR" (at 33.02 200.66 180) (fields_autoplaced) (effects (font (size 1.27 1.27)) (justify right bottom)))
+  (label "LDR_SENSE" (at 48.26 215.90 0) (fields_autoplaced) (effects (font (size 1.27 1.27)) (justify left bottom)))
+  (text "Light sensor (switched by D7), RV1 sets dusk" (at 20.32 195.58 0) (effects (font (size 1.27 1.27) (thickness 0.1524)) (justify left bottom)))
   (label "BTN" (at 88.90 213.36 180) (fields_autoplaced) (effects (font (size 1.27 1.27)) (justify right bottom)))
   (text "Test button" (at 83.82 195.58 0) (effects (font (size 1.27 1.27) (thickness 0.1524)) (justify left bottom)))
@@
   (wire (pts (xy 119.38 162.56) (xy 129.54 162.56)) (stroke (width 0) (type default)))
   (wire (pts (xy 119.38 165.10) (xy 129.54 165.10)) (stroke (width 0) (type default)))
-  (wire (pts (xy 33.02 203.20) (xy 40.64 203.20)) (stroke (width 0) (type default)))
-  (wire (pts (xy 40.64 203.20) (xy 40.64 208.28)) (stroke (width 0) (type default)))
-  (wire (pts (xy 40.64 215.90) (xy 40.64 218.44)) (stroke (width 0) (type default)))
-  (wire (pts (xy 40.64 218.44) (xy 40.64 223.52)) (stroke (width 0) (type default)))
-  (wire (pts (xy 40.64 218.44) (xy 48.26 218.44)) (stroke (width 0) (type default)))
-  (wire (pts (xy 40.64 231.14) (xy 40.64 236.22)) (stroke (width 0) (type default)))
+  (wire (pts (xy 33.02 200.66) (xy 40.64 200.66)) (stroke (width 0) (type default)))
+  (wire (pts (xy 40.64 200.66) (xy 40.64 205.74)) (stroke (width 0) (type default)))
+  (wire (pts (xy 40.64 213.36) (xy 40.64 215.90)) (stroke (width 0) (type default)))
+  (wire (pts (xy 40.64 215.90) (xy 40.64 217.17)) (stroke (width 0) (type default)))
+  (wire (pts (xy 40.64 215.90) (xy 48.26 215.90)) (stroke (width 0) (type default)))
+  (wire (pts (xy 40.64 224.79) (xy 40.64 229.87)) (stroke (width 0) (type default)))
+  (wire (pts (xy 44.45 233.68) (xy 46.99 233.68)) (stroke (width 0) (type default)))
+  (wire (pts (xy 46.99 233.68) (xy 46.99 238.76)) (stroke (width 0) (type default)))
+  (wire (pts (xy 46.99 238.76) (xy 40.64 238.76)) (stroke (width 0) (type default)))
+  (wire (pts (xy 40.64 237.49) (xy 40.64 238.76)) (stroke (width 0) (type default)))
   (wire (pts (xy 88.90 213.36) (xy 96.52 213.36)) (stroke (width 0) (type default)))
   (wire (pts (xy 106.68 213.36) (xy 111.76 213.36)) (stroke (width 0) (type default)))
@@
   (junction (at 137.16 104.14) (diameter 0) (color 0 0 0 0))
   (junction (at 236.22 50.80) (diameter 0) (color 0 0 0 0))
-  (junction (at 40.64 218.44) (diameter 0) (color 0 0 0 0))
+  (junction (at 40.64 215.90) (diameter 0) (color 0 0 0 0))
   (junction (at 208.28 170.18) (diameter 0) (color 0 0 0 0))
   (junction (at 238.76 165.10) (diameter 0) (color 0 0 0 0))
@@
     (in_bom yes) (on_board yes) (dnp no)
     (property "Reference" "R3" (at 306.07 46.99 90) (effects (font (size 1.27 1.27))))
-    (property "Value" "47R" (at 306.07 54.61 90) (effects (font (size 1.27 1.27))))
+    (property "Value" "56R" (at 306.07 54.61 90) (effects (font (size 1.27 1.27))))
     (property "Footprint" "Resistor_THT:R_Axial_DIN0207_L6.3mm_D2.5mm_P10.16mm_Horizontal" (at 306.07 50.80 0) (effects (font (size 1.27 1.27)) hide))
     (property "Datasheet" "~" (at 306.07 50.80 0) (effects (font (size 1.27 1.27)) hide))
-    (property "Note" "low-power string only; model ~15 mA @3.7 V, 56R if >22 mA @4.2 V" (at 306.07 56.80 90) (effects (font (size 1.016 1.016) italic)))
+    (property "Note" "low-power string only; model ~13 mA @3.7 V, 68R if >20 mA @4.2 V" (at 306.07 56.80 90) (effects (font (size 1.016 1.016) italic)))
     (pin "1")
     (pin "2")
@@
     (instances (project "SolarLights_Lite" (path "/f1c127e7-0661-5259-aeb4-1ed89663ebe4" (reference "M2") (unit 1))))
   )
-  (symbol (lib_id "SolarLights_Lite:LDR") (at 40.64 212.09 0) (unit 1)
-    (in_bom yes) (on_board yes) (dnp no)
-    (property "Reference" "LDR1" (at 43.18 210.82 0) (effects (font (size 1.27 1.27)) (justify left)))
-    (property "Value" "LDR" (at 43.18 213.36 0) (effects (font (size 1.27 1.27)) (justify left)))
-    (property "Footprint" "" (at 40.64 212.09 0) (effects (font (size 1.27 1.27)) hide))
-    (property "Datasheet" "~" (at 40.64 212.09 0) (effects (font (size 1.27 1.27)) hide))
+  (symbol (lib_id "SolarLights_Lite:LDR") (at 40.64 209.55 0) (unit 1)
+    (in_bom yes) (on_board yes) (dnp no)
+    (property "Reference" "LDR1" (at 43.18 208.28 0) (effects (font (size 1.27 1.27)) (justify left)))
+    (property "Value" "LDR" (at 43.18 210.82 0) (effects (font (size 1.27 1.27)) (justify left)))
+    (property "Footprint" "" (at 40.64 209.55 0) (effects (font (size 1.27 1.27)) hide))
+    (property "Datasheet" "~" (at 40.64 209.55 0) (effects (font (size 1.27 1.27)) hide))
     (pin "1")
     (pin "2")
     (instances (project "SolarLights_Lite" (path "/f1c127e7-0661-5259-aeb4-1ed89663ebe4" (reference "LDR1") (unit 1))))
   )
-  (symbol (lib_id "Device:R") (at 40.64 227.33 0) (unit 1)
-    (in_bom yes) (on_board yes) (dnp no)
-    (property "Reference" "R4" (at 43.18 226.06 0) (effects (font (size 1.27 1.27)) (justify left)))
-    (property "Value" "47k" (at 43.18 228.60 0) (effects (font (size 1.27 1.27)) (justify left)))
-    (property "Footprint" "Resistor_THT:R_Axial_DIN0207_L6.3mm_D2.5mm_P10.16mm_Horizontal" (at 40.64 227.33 0) (effects (font (size 1.27 1.27)) hide))
-    (property "Datasheet" "~" (at 40.64 227.33 0) (effects (font (size 1.27 1.27)) hide))
+  (symbol (lib_id "Device:R") (at 40.64 220.98 0) (unit 1)
+    (in_bom yes) (on_board yes) (dnp no)
+    (property "Reference" "R4" (at 43.18 219.71 0) (effects (font (size 1.27 1.27)) (justify left)))
+    (property "Value" "22k" (at 43.18 222.25 0) (effects (font (size 1.27 1.27)) (justify left)))
+    (property "Footprint" "Resistor_THT:R_Axial_DIN0207_L6.3mm_D2.5mm_P10.16mm_Horizontal" (at 40.64 220.98 0) (effects (font (size 1.27 1.27)) hide))
+    (property "Datasheet" "~" (at 40.64 220.98 0) (effects (font (size 1.27 1.27)) hide))
     (pin "1")
     (pin "2")
     (instances (project "SolarLights_Lite" (path "/f1c127e7-0661-5259-aeb4-1ed89663ebe4" (reference "R4") (unit 1))))
   )
+  (symbol (lib_id "Device:R_Potentiometer") (at 40.64 233.68 0) (unit 1)
+    (in_bom yes) (on_board yes) (dnp no)
+    (property "Reference" "RV1" (at 48.26 232.41 0) (effects (font (size 1.27 1.27)) (justify left)))
+    (property "Value" "50k trim" (at 48.26 234.95 0) (effects (font (size 1.27 1.27)) (justify left)))
+    (property "Footprint" "Potentiometer_THT:Potentiometer_Bourns_3296W_Vertical" (at 40.64 233.68 0) (effects (font (size 1.27 1.27)) hide))
+    (property "Datasheet" "~" (at 40.64 233.68 0) (effects (font (size 1.27 1.27)) hide))
+    (property "Note" "3296W; wiper to pin 3" (at 48.26 236.98 0) (effects (font (size 1.016 1.016) italic) (justify left)))
+    (pin "1")
+    (pin "2")
+    (pin "3")
+    (instances (project "SolarLights_Lite" (path "/f1c127e7-0661-5259-aeb4-1ed89663ebe4" (reference "RV1") (unit 1))))
+  )
   (symbol (lib_id "Switch:SW_Push") (at 101.60 213.36 0) (unit 1)
     (in_bom yes) (on_board yes) (dnp no)
     (property "Reference" "SW1" (at 101.60 209.55 0) (effects (font (size 1.27 1.27))))
-    (property "Value" "test" (at 101.60 215.90 0) (effects (font (size 1.27 1.27))))
+    (property "Value" "TEST" (at 101.60 215.90 0) (effects (font (size 1.27 1.27))))
     (property "Footprint" "" (at 101.60 213.36 0) (effects (font (size 1.27 1.27)) hide))
     (property "Datasheet" "~" (at 101.60 213.36 0) (effects (font (size 1.27 1.27)) hide))
@@
     (instances (project "SolarLights_Lite" (path "/f1c127e7-0661-5259-aeb4-1ed89663ebe4" (reference "#PWR106") (unit 1))))
   )
-  (symbol (lib_id "power:GND") (at 40.64 236.22 0) (unit 1)
-    (in_bom yes) (on_board yes) (dnp no)
-    (property "Reference" "#PWR107" (at 43.18 234.95 0) (effects (font (size 1.27 1.27)) hide (justify left)))
-    (property "Value" "GND" (at 43.18 237.49 0) (effects (font (size 1.27 1.27)) hide (justify left)))
-    (property "Footprint" "" (at 40.64 236.22 0) (effects (font (size 1.27 1.27)) hide))
-    (property "Datasheet" "~" (at 40.64 236.22 0) (effects (font (size 1.27 1.27)) hide))
+  (symbol (lib_id "power:GND") (at 40.64 238.76 0) (unit 1)
+    (in_bom yes) (on_board yes) (dnp no)
+    (property "Reference" "#PWR107" (at 43.18 237.49 0) (effects (font (size 1.27 1.27)) hide (justify left)))
+    (property "Value" "GND" (at 43.18 240.03 0) (effects (font (size 1.27 1.27)) hide (justify left)))
+    (property "Footprint" "" (at 40.64 238.76 0) (effects (font (size 1.27 1.27)) hide))
+    (property "Datasheet" "~" (at 40.64 238.76 0) (effects (font (size 1.27 1.27)) hide))
     (pin "1")
     (instances (project "SolarLights_Lite" (path "/f1c127e7-0661-5259-aeb4-1ed89663ebe4" (reference "#PWR107") (unit 1))))
