File: hardware/pcb-rev-c/SolarLights_Carrier_RevC.kicad_sch (KiCad schematic)
At the start: 27 parts, among them M1 TP4056 module, Q2 2N3904 / EBC

Commit message: feat(pcb): carrier Rev C with LDR trim, TEST button and box-header ISP
R3 56R, R4 22k + RV1 50k 3296W rheostat, on-board 6x6 TEST switch, sideways
ISP with optional DC3-6P box header, name and repo on silkscreen. Docs 01-13,
drawings, layouts, netlist, KiCad schematic and renders follow Rev C.
Parts:
- removed JBUTTON1: SW1 D2 / -, Carrier:SolderPads_1x02_P2.54mm, symbol Connector_Generic:Conn_01x02
- added RV1: 50k 3296W, Carrier:Potentiometer_Bourns_3296W_Vertical, symbol Device:R_Potentiometer
- added SW1: 6x6 tactile, Carrier:SW_PUSH_6mm_H9.5mm, symbol Switch:SW_Push
- JISP1: value ISP -> 2x3 male header 2.54 mm; footprint Carrier:Pads_2x03_P2.54mm -> Carrier:IDC-Header_2x03_P2.54mm_Vertical
- R3: value 47R / 0.25W -> 56R / 0.25W
- R4: value 47k -> 22k
Connections:
- net GND_LOAD: now also RV1.2, RV1.3, SW1.2; no longer R4.2
- net TEST: now also SW1.1
- new net LDR_TRIM: R4.2, RV1.1
Other:
- note added: "R3 56R (was 47R in Rev B): about 19 mA peak at 4.2 V, still to confirm on the bench. No LED-cable short protection."
- note added: "RV1 50k rheostat + R4 22k = LDR lower leg 22k-72k; mid-travel matches the Rev B 47k. SW1 is on the board."
- note removed: "R3 peak current requires bench qualification. 47R matches existing circuit; no LED-cable short protection."
Changed lines of the file:
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@@
 (label "GND_LOAD" (at 76.2 143.51 0) (effects (font (size 1 1)) (justify left bottom)))
 (symbol (lib_id "Device:R") (at 30.48 186.69 0) (unit 1) (in_bom yes) (on_board yes) (dnp no) (property "Reference" "R3" (at 30.48 176.88 0) (effects (font (size 1.27 1.27))))
-(property "Value" "47R / 0.25W" (at 30.48 179.88 0) (effects (font (size 0.95 0.95))))
+(property "Value" "56R / 0.25W" (at 30.48 179.88 0) (effects (font (size 0.95 0.95))))
 (property "Footprint" "Carrier:R_Axial_DIN0207_L6.3mm_D2.5mm_P7.62mm_Horizontal" (at 30.48 186.69 0) (effects (font (size 1.27 1.27)) hide))
 (property "Datasheet" "" (at 30.48 186.69 0) (effects (font (size 1.27 1.27)) hide)) (pin "1") (pin "2")(instances (project "SolarLights_Carrier_RevC" (path "/b93d1bc0-78a9-5637-b0dd-81c4f0127b80" (reference "R3") (unit 1)))))
@@
 (label "LDR_SENSE" (at 93.98 189.23 180) (effects (font (size 1 1)) (justify right bottom)))
 (symbol (lib_id "Device:R") (at 143.51 186.69 0) (unit 1) (in_bom yes) (on_board yes) (dnp no) (property "Reference" "R4" (at 143.51 176.88 0) (effects (font (size 1.27 1.27))))
-(property "Value" "47k" (at 143.51 179.88 0) (effects (font (size 0.95 0.95))))
+(property "Value" "22k" (at 143.51 179.88 0) (effects (font (size 0.95 0.95))))
 (property "Footprint" "Carrier:R_Axial_DIN0207_L6.3mm_D2.5mm_P7.62mm_Horizontal" (at 143.51 186.69 0) (effects (font (size 1.27 1.27)) hide))
 (property "Datasheet" "" (at 143.51 186.69 0) (effects (font (size 1.27 1.27)) hide)) (pin "1") (pin "2")(instances (project "SolarLights_Carrier_RevC" (path "/b93d1bc0-78a9-5637-b0dd-81c4f0127b80" (reference "R4") (unit 1)))))
@@
 (label "LDR_SENSE" (at 153.67 182.88 0) (effects (font (size 1 1)) (justify left bottom)))
 (wire (pts (xy 143.51 190.5) (xy 153.67 190.5)) (stroke (width 0) (type default)))
-(label "GND_LOAD" (at 153.67 190.5 0) (effects (font (size 1 1)) (justify left bottom)))
-(symbol (lib_id "Connector_Generic:Conn_01x02") (at 143.51 227.33 0) (unit 1) (in_bom yes) (on_board yes) (dnp no) (property "Reference" "JBUTTON1" (at 143.51 221.33 0) (effects (font (size 1.27 1.27))))
-(property "Value" "SW1 D2 / -" (at 143.51 224.33 0) (effects (font (size 0.95 0.95))))
-(property "Footprint" "Carrier:SolderPads_1x02_P2.54mm" (at 143.51 227.33 0) (effects (font (size 1.27 1.27)) hide))
-(property "Datasheet" "" (at 143.51 227.33 0) (effects (font (size 1.27 1.27)) hide)) (pin "1") (pin "2")(instances (project "SolarLights_Carrier_RevC" (path "/b93d1bc0-78a9-5637-b0dd-81c4f0127b80" (reference "JBUTTON1") (unit 1)))))
+(label "LDR_TRIM" (at 153.67 190.5 0) (effects (font (size 1 1)) (justify left bottom)))
+(symbol (lib_id "Device:R_Potentiometer") (at 160.02 204.47 0) (unit 1) (in_bom yes) (on_board yes) (dnp no) (property "Reference" "RV1" (at 160.02 194.66 0) (effects (font (size 1.27 1.27))))
+(property "Value" "50k 3296W" (at 160.02 197.66 0) (effects (font (size 0.95 0.95))))
+(property "Footprint" "Carrier:Potentiometer_Bourns_3296W_Vertical" (at 160.02 204.47 0) (effects (font (size 1.27 1.27)) hide))
+(property "Datasheet" "" (at 160.02 204.47 0) (effects (font (size 1.27 1.27)) hide)) (pin "1") (pin "2") (pin "3")(instances (project "SolarLights_Carrier_RevC" (path "/b93d1bc0-78a9-5637-b0dd-81c4f0127b80" (reference "RV1") (unit 1)))))
+(wire (pts (xy 160.02 200.66) (xy 170.18 200.66)) (stroke (width 0) (type default)))
+(label "LDR_TRIM" (at 170.18 200.66 0) (effects (font (size 1 1)) (justify left bottom)))
+(wire (pts (xy 163.83 204.47) (xy 173.99 204.47)) (stroke (width 0) (type default)))
+(label "GND_LOAD" (at 173.99 204.47 0) (effects (font (size 1 1)) (justify left bottom)))
+(wire (pts (xy 160.02 208.28) (xy 170.18 208.28)) (stroke (width 0) (type default)))
+(label "GND_LOAD" (at 170.18 208.28 0) (effects (font (size 1 1)) (justify left bottom)))
+(symbol (lib_id "Switch:SW_Push") (at 143.51 227.33 0) (unit 1) (in_bom yes) (on_board yes) (dnp no) (property "Reference" "SW1" (at 143.51 221.33 0) (effects (font (size 1.27 1.27))))
+(property "Value" "6x6 tactile" (at 143.51 224.33 0) (effects (font (size 0.95 0.95))))
+(property "Footprint" "Carrier:SW_PUSH_6mm_H9.5mm" (at 143.51 227.33 0) (effects (font (size 1.27 1.27)) hide))
+(property "Datasheet" "" (at 143.51 227.33 0) (effects (font (size 1.27 1.27)) hide)) (pin "1") (pin "2")(instances (project "SolarLights_Carrier_RevC" (path "/b93d1bc0-78a9-5637-b0dd-81c4f0127b80" (reference "SW1") (unit 1)))))
 (wire (pts (xy 138.43 227.33) (xy 128.27 227.33)) (stroke (width 0) (type default)))
 (label "TEST" (at 128.27 227.33 180) (effects (font (size 1 1)) (justify right bottom)))
-(wire (pts (xy 138.43 229.87) (xy 128.27 229.87)) (stroke (width 0) (type default)))
-(label "GND_LOAD" (at 128.27 229.87 180) (effects (font (size 1 1)) (justify right bottom)))
+(wire (pts (xy 148.59 227.33) (xy 158.75 227.33)) (stroke (width 0) (type default)))
+(label "GND_LOAD" (at 158.75 227.33 0) (effects (font (size 1 1)) (justify left bottom)))
 (symbol (lib_id "Device:R") (at 184.15 185.42000000000002 0) (unit 1) (in_bom yes) (on_board yes) (dnp no) (property "Reference" "R5" (at 184.15 175.61 0) (effects (font (size 1.27 1.27))))
 (property "Value" "220k" (at 184.15 178.61 0) (effects (font (size 0.95 0.95))))
@@
 (no_connect (at 87.63 109.22))
 (symbol (lib_id "Connector_Generic:Conn_02x03_Odd_Even") (at 124.46000000000001 93.98 0) (unit 1) (in_bom yes) (on_board yes) (dnp no) (property "Reference" "JISP1" (at 124.46000000000001 85.44 0) (effects (font (size 1.27 1.27))))
-(property "Value" "ISP" (at 124.46000000000001 88.44 0) (effects (font (size 0.95 0.95))))
-(property "Footprint" "Carrier:Pads_2x03_P2.54mm" (at 124.46000000000001 93.98 0) (effects (font (size 1.27 1.27)) hide))
+(property "Value" "2x3 male header 2.54 mm" (at 124.46000000000001 88.44 0) (effects (font (size 0.95 0.95))))
+(property "Footprint" "Carrier:IDC-Header_2x03_P2.54mm_Vertical" (at 124.46000000000001 93.98 0) (effects (font (size 1.27 1.27)) hide))
 (property "Datasheet" "" (at 124.46000000000001 93.98 0) (effects (font (size 1.27 1.27)) hide)) (pin "1") (pin "2") (pin "3") (pin "4") (pin "5") (pin "6")(instances (project "SolarLights_Carrier_RevC" (path "/b93d1bc0-78a9-5637-b0dd-81c4f0127b80" (reference "JISP1") (unit 1)))))
 (wire (pts (xy 119.38 91.44) (xy 109.22 91.44)) (stroke (width 0) (type default)))
@@
 (text "U0 solar buck, U3 buck-boost, cells and S1 are external. B- is its own net: never joined to GND_LOAD. No fuses. All returns = M1 OUT-." (at 201 253 0) (effects (font (size 1.3 1.3))))
 (text "Tier 0: omit telemetry. Tier 1: JP1 OPEN, USB. Tier 2: JP1 + JP2 closed, NO USB. JP3 closed only with powered M3." (at 201 260 0) (effects (font (size 1.3 1.3))))
-(text "R3 peak current requires bench qualification. 47R matches existing circuit; no LED-cable short protection." (at 201 267 0) (effects (font (size 1.3 1.3)))))
+(text "R3 56R (was 47R in Rev B): about 19 mA peak at 4.2 V, still to confirm on the bench. No LED-cable short protection." (at 201 267 0) (effects (font (size 1.3 1.3))))
+(text "RV1 50k rheostat + R4 22k = LDR lower leg 22k-72k; mid-travel matches the Rev B 47k. SW1 is on the board." (at 201 274 0) (effects (font (size 1.3 1.3)))))
